Commit message: Port URDF generation to the CAD wrist bracket
The merge from main brought in URDF generation (PR #5) written against the
old inline-box bracket spec (WRIST_BRACKET_BOXES on the link6 bodies), which
no longer exists: the bracket is now the user-authored CAD STL plus screw
and standoff cylinders, rigid to the link5 forearm bodies. CI failed
collecting tests/test_urdf_generation.py on the missing import.

The URDF now carries the same bracket as the MJCF: the STL mesh visual
(assets/anvil_wrist_bracket.stl, right side mirrored via a negative y
scale), the four dark screw heads, and the forearm standoff as cylinder
visuals on the link5 links, with both materials declared at the robot root.
Tests assert the mesh reference/scale, every cylinder's midpoint, length,
radius, axis orientation, and material against the spec, and the mesh-path
test accepts the models/assets reference alongside the upstream submodule
paths.

Co-Authored-By: Claude Fable 5 <noreply@anthropic.com>

File: models/anvil_openarm_bimanual.urdf (robot description, URDF)
Before this commit: robot anvil_openarm_v20, 24 links, 23 joints
Links:
- link openarm_left_link5: geometry collision mesh filename=../upstream/openarm_description/assets/robot/openarm_v2.0/m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 scale=1 -1 1; visual cylinder length=0.003999999999999997 radius=0.003
- link openarm_left_link6: geometry collision mesh filename=../upstream/openarm_description/assets/robot/openarm_v2.0/m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 scale=1 -1 1; visual mesh filename=../upstream/openarm_description/assets/robot/openarm_v2.0/m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 scale=1 -1 1
- link openarm_right_link5: geometry collision mesh filename=../upstream/openarm_description/assets/robot/openarm_v2.0/m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 scale=1 1 1; visual cylinder length=0.003999999999999997 radius=0.003
- link openarm_right_link6: geometry collision mesh filename=../upstream/openarm_description/assets/robot/openarm_v2.0/m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 scale=1 1 1; visual mesh filename=../upstream/openarm_description/assets/robot/openarm_v2.0/m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 scale=1 1 1
