Commit message: Correct side-specific Anvil joint limits

File: models/anvil_openarm_bimanual.urdf (robot description, URDF)
Before this commit: robot anvil_openarm_v20, 24 links, 23 joints
Joints:
- joint openarm_left_joint1: limit lower=-2.3562 upper=2.3562 effort=40 velocity=16.755 -> lower=-3.4907 upper=1.3963 effort=40 velocity=16.755
- joint openarm_right_joint1: limit lower=-2.3562 upper=2.3562 effort=40 velocity=16.755 -> lower=-1.3963 upper=3.4907 effort=40 velocity=16.755
- joint openarm_right_joint6: limit lower=-0.7854 upper=1.2217 effort=7 velocity=20.944 -> lower=-1.2217 upper=0.7854 effort=7 velocity=20.944
